File: Eagle/Hoverboard JC2015.7.31.brd (EAGLE design)
At the start: 130.3 x 58.4 mm, 178 parts, among them IC1 7805DT, IC2 LD1117S33, IC3 MPU-6881, IC4 LM358D, IC5 EG1182, J1 L-KLS1-2.50L-03-S, J2 L-KLS1-2.50L-02-S, J3 HALL, J5 USART, J6 LED, J7 L-KLS1-2.50L-02-S, J8 L-KLS1-2.50L-02-S, Q1 1013, Q10 SS8550, Q11 SS8050, Q12 SS8050, Q13 110N8F6, Q14 2N5551, Q15 SS8550, Q16 SS8550, Q17 110N8F6, Q18 SS8550, Q19 SS8050, Q2 MJD41C, Q20 SS8050, Q21 110N8F6, Q22 2N5551, Q23 SS8550, Q24 SS8550, Q25 110N8F6, Q26 SS8550, Q27 SS8050, Q28 SS8050, Q29 110N8F6, Q6 2N5551, Q7 SS8550, Q8 SS8550, Q9 110N8F6, U1 GD32F103C8T6

Commit message: Reworked schematics
Parts:
- J4: value (none) -> External
- J9: value (none) -> Programming
Connections:
- net GNDI renamed V-CURRENTSHUNT
- net N$18 renamed PC14
- net N$49 renamed PC13
Changed lines of the file:
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@@
 <attribute name="VALUE" x="67.168" y="6.655" locked="yes" size="1.27" layer="27"/>
 </element>
-<element name="J4" library="JohMah" package="FE06-1" value="" x="56.25" y="5.08" locked="yes" smashed="yes">
+<element name="J4" library="JohMah" package="FE06-1" value="External" x="56.25" y="5.08" locked="yes" smashed="yes">
 <attribute name="NAME" x="49.011" y="2.413" locked="yes" size="1.27" layer="25" ratio="10"/>
 <attribute name="VALUE" x="48.63" y="2.159" locked="yes" size="1.27" layer="27" ratio="10"/>
 </element>
-<element name="J9" library="JohMah" package="FE04-1" value="" x="32.639" y="27.051" locked="yes" smashed="yes" rot="R180">
+<element name="J9" library="JohMah" package="FE04-1" value="Programming" x="32.639" y="27.051" locked="yes" smashed="yes" rot="R180">
 <attribute name="NAME" x="33.19" y="25.46" locked="yes" size="1.27" layer="25" rot="R180"/>
 <attribute name="VALUE" x="38.239" y="25.476" locked="yes" size="1.27" layer="27" rot="R180"/>
@@
 <contactref element="J4" pad="6"/>
 <contactref element="J5" pad="4"/>
+<contactref element="Q31" pad="E"/>
 <contactref element="J1" pad="1"/>
-<contactref element="Q31" pad="E"/>
 <wire x1="113.919" y1="31.877" x2="116.84" y2="47.74" width="0" layer="19" extent="1-1"/>
 <wire x1="106.807" y1="25.847" x2="113.919" y2="31.877" width="0" layer="19" extent="1-1"/>
@@
 <wire x1="108.966" y1="21.021" x2="113.919" y2="21.717" width="0" layer="19" extent="1-1"/>
 </signal>
-<signal name="N$18">
+<signal name="PC14">
 <contactref element="OK1" pad="3"/>
 <contactref element="R15" pad="1"/>
+<contactref element="R16" pad="2"/>
 <contactref element="U1" pad="3"/>
-<contactref element="R16" pad="2"/>
 <wire x1="106.807" y1="27.747" x2="111.379" y2="31.877" width="0" layer="19" extent="1-1"/>
 <wire x1="108.966" y1="25.847" x2="106.807" y2="27.747" width="0" layer="19" extent="1-1"/>
@@
 <wire x1="18.923" y1="21.336" x2="27.94" y2="16.83" width="0" layer="19" extent="1-1"/>
 </signal>
-<signal name="N$49">
+<signal name="PC13">
 <contactref element="OK2" pad="3"/>
-<contactref element="U1" pad="2"/>
 <contactref element="R61" pad="1"/>
 <contactref element="R60" pad="2"/>
+<contactref element="U1" pad="2"/>
 <wire x1="38.1" y1="16.19" x2="41.47" y2="23.205" width="0" layer="19" extent="1-1"/>
-<wire x1="20.32" y1="26.99" x2="41.47" y2="23.205" width="0" layer="19" extent="1-1"/>
+<wire x1="20.32" y1="26.99" x2="38.1" y2="16.19" width="0" layer="19" extent="1-1"/>
 <wire x1="16.383" y1="31.496" x2="20.32" y2="26.99" width="0" layer="19" extent="1-1"/>
 </signal>
@@
 <wire x1="80.264" y1="40.325" x2="77.597" y2="42.121" width="0" layer="19" extent="1-1"/>
 </signal>
-<signal name="GNDI">
-<contactref element="Q12" pad="E"/>
-<contactref element="Q13" pad="S"/>
-<contactref element="C39" pad="1"/>
-<contactref element="R1" pad="2"/>
-<contactref element="Q20" pad="E"/>
-<contactref element="Q21" pad="S"/>
-<contactref element="C46" pad="1"/>
-<contactref element="Q28" pad="E"/>
-<contactref element="Q29" pad="S"/>
-<contactref element="C53" pad="1"/>
-<contactref element="R44" pad="2"/>
-<wire x1="116.84" y1="42.33" x2="116.84" y2="53.34" width="0" layer="19" extent="1-1"/>
-<wire x1="78.547" y1="39.921" x2="116.84" y2="42.33" width="0" layer="19" extent="1-1"/>
-<wire x1="75.438" y1="47.752" x2="78.547" y2="39.921" width="0" layer="19" extent="1-1"/>
-<wire x1="66.736" y1="27.432" x2="78.547" y2="39.921" width="0" layer="19" extent="1-1"/>
-<wire x1="46.162" y1="39.794" x2="66.736" y2="27.432" width="0" layer="19" extent="1-1"/>
-<wire x1="43.473" y1="44.45" x2="46.162" y2="39.794" width="0" layer="19" extent="1-1"/>
-<wire x1="46.228" y1="47.752" x2="43.473" y2="44.45" width="0" layer="19" extent="1-1"/>
-<wire x1="19.238" y1="39.413" x2="43.473" y2="44.45" width="0" layer="19" extent="1-1"/>
-<wire x1="17.184" y1="44.323" x2="19.238" y2="39.413" width="0" layer="19" extent="1-1"/>
-<wire x1="16.891" y1="47.752" x2="17.184" y2="44.323" width="0" layer="19" extent="1-1"/>
-</signal>
 <signal name="N$69">
 <contactref element="R75" pad="1"/>
@@
 <wire x1="2.28" y1="55.88" x2="12.192" y2="49.316" width="0" layer="19" extent="1-1"/>
 </signal>
+<signal name="V-CURRENTSHUNT">
+<contactref element="Q12" pad="E"/>
+<contactref element="Q13" pad="S"/>
+<contactref element="C39" pad="1"/>
+<contactref element="Q20" pad="E"/>
+<contactref element="Q21" pad="S"/>
+<contactref element="C46" pad="1"/>
+<contactref element="Q28" pad="E"/>
+<contactref element="Q29" pad="S"/>
+<contactref element="C53" pad="1"/>
+<contactref element="R1" pad="2"/>
+<contactref element="R44" pad="2"/>
+<wire x1="116.84" y1="42.33" x2="116.84" y2="53.34" width="0" layer="19" extent="1-1"/>
+<wire x1="78.547" y1="39.921" x2="116.84" y2="42.33" width="0" layer="19" extent="1-1"/>
+<wire x1="75.438" y1="47.752" x2="78.547" y2="39.921" width="0" layer="19" extent="1-1"/>
+<wire x1="66.736" y1="27.432" x2="78.547" y2="39.921" width="0" layer="19" extent="1-1"/>
+<wire x1="46.162" y1="39.794" x2="66.736" y2="27.432" width="0" layer="19" extent="1-1"/>
+<wire x1="43.473" y1="44.45" x2="46.162" y2="39.794" width="0" layer="19" extent="1-1"/>
+<wire x1="46.228" y1="47.752" x2="43.473" y2="44.45" width="0" layer="19" extent="1-1"/>
+<wire x1="19.238" y1="39.413" x2="43.473" y2="44.45" width="0" layer="19" extent="1-1"/>
+<wire x1="17.184" y1="44.323" x2="19.238" y2="39.413" width="0" layer="19" extent="1-1"/>
+<wire x1="16.891" y1="47.752" x2="17.184" y2="44.323" width="0" layer="19" extent="1-1"/>
+</signal>
 </signals>
