File: Eagle/Hoverboard JC2015.7.31.sch (EAGLE design)
At the start: 178 parts, among them IC1 7805DT, IC2 LD1117S33, IC3 MPU-6881, IC4 LM358D, IC5 EG1182, J1 L-KLS1-2.50L-03-S, J2 L-KLS1-2.50L-02-S, J3 HALL, J5 USART, J6 LED, J7 L-KLS1-2.50L-02-S, J8 L-KLS1-2.50L-02-S, Q1 1013, Q10 SS8550, Q11 SS8050, Q12 SS8050, Q13 110N8F6, Q14 2N5551, Q15 SS8550, Q16 SS8550, Q17 110N8F6, Q18 SS8550, Q19 SS8050, Q2 MJD41C, Q20 SS8050, Q21 110N8F6, Q22 2N5551, Q23 SS8550, Q24 SS8550, Q25 110N8F6, Q26 SS8550, Q27 SS8050, Q28 SS8050, Q29 110N8F6, Q6 2N5551, Q7 SS8550, Q8 SS8550, Q9 110N8F6, U1 GD32F103C8T6

Commit message: Reworked schematics
Parts:
- J4: value (none) -> External
- J9: value (none) -> Programming
Connections:
- net GNDI renamed V-CURRENTSHUNT
- net N$18 renamed PC14
- net N$49 renamed PC13
- net PA10: now also U1A.PA10/TIMER0_CH2; no longer U1A.PA10
- net PA13: now also U1A.PA13/JTMS:SWDIO; no longer U1A.PA13
- net PA14: now also U1A.PA14/JTMS:SWCLK; no longer U1A.PA14
- net PA5: now also U1A.PA5/ADC01_IN5; no longer U1A.PA5
- net PA6: now also U1A.PA6/ADC01_IN6; no longer U1A.PA6
- net PA7: now also U1A.PA7/ADC01_IN7; no longer U1A.PA7
- net PA8: now also U1A.PA8/TIMER0_CH0; no longer U1A.PA8
- net PA9: now also U1A.PA9/TIMER0_CH1; no longer U1A.PA9
- net PB0: now also U1A.PB0/ADC01_IN8; no longer U1A.PB0
- net PB10: now also U1A.PB10/USART2_TX; no longer U1A.PB10
- net PB11: now also U1A.PB11/USART2-RX; no longer U1A.PB11
- net PB12: now also U1A.PB12/TIMER0_BRKIN; no longer U1A.PB12
- net PB13: now also U1A.PB13/TIMER0_CH0_ON; no longer U1A.PB13
- net PB14: now also U1A.PB14/TIMER0_CH1_ON; no longer U1A.PB14
- net PB15: now also U1A.PB15/TIMER0_CH2_ON; no longer U1A.PB15
- net PB4: now also U1A.PB4/SPI0_MISO; no longer U1A.PB4
- net PB5: now also U1A.PB5/SPI0_MOSI; no longer U1A.PB5
- net PB6: now also U1A.PB6/USART0_TX; no longer U1A.PB6
- net PB7: now also U1A.PB7/USART0_RX; no longer U1A.PB7
- net PB8: now also U1A.PB8/I2C0_SCL; no longer U1A.PB8
- net PB9: now also U1A.PB9/I2C0_SDA; no longer U1A.PB9
Other:
- moved on the sheet: IC4A, OK1, OK2, R1, R14, R15, R16, R32, R34, R35, R44, R53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
